File: untitled.brd (EAGLE design)
At the start: 100 x 100 mm, 23 parts, among them K1 SLA-12VDC-SL-C, T1 BC547, X2 pzem-004t

Commit message: comit
comit
Parts:
- removed D1: 1N4004, diode:DO41-10
- removed K1: SLA-12VDC-SL-C, SLA-12VDC-SL-C:RELAY_SLA-12VDC-SL-C
- removed LED1: (no value), led:LED5MM
- removed OK1: PC817, optocoupler:DIL04
- removed R1: 1k, rcl:0207/15
- removed R2: 330, rcl:0207/15
- removed RELAY: KF76, kf76:KF76
- removed T1: BC547, transistor:TO92
- added LCD1: LCD_2X16_SIL, lcd_2x16_led_backlight:HY-1602F
Connections:
- removed net N$11: K1.NC, RELAY.P$1
- removed net N$18: LED1.A, R2.1
- removed net N$19: OK1.2, R2.2
- removed net N$2: OK1.3, R1.1
- removed net N$20: LED1.K, NODE1.D7
- removed net N$3: R1.2, T1.2
- removed net N$5: D1.A, K1.C2, T1.3
- removed net N$8: K1.COM1, K1.COM2
- new net VSS: LCD1.1
- net 3V: no longer NODE1.3V3@2, OK1.1
- net 3V3: now also NODE1.3V3@2
- net GND: no longer T1.1
- net N$7: no longer RELAY.P$2
- net VCC: now also LCD1.2; no longer D1.C, K1.C1, OK1.4
Routing:
- net VCC: track 298.5 -> 36.9 mm
- net N$11: track 122.4 -> 0.00 mm
- net GND: track 162.2 -> 69.3 mm
- net 3V: track 128.1 -> 65.7 mm
- net N$8: track 60.6 -> 0.00 mm
- net N$20: track 43.8 -> 0.00 mm
- net N$2: track 22.5 -> 0.00 mm
- net N$3: track 17.8 -> 0.00 mm
- net N$5: track 17.6 -> 0.00 mm
- net N$18: track 15.7 -> 0.00 mm
- net N$7: track 203.5 -> 195.4 mm
- net N$19: track 7.81 -> 0.00 mm

Commit message: 0021
Parts:
- moved LCD1 75.7 mm to (13.2, 37.8), turned to 0 degrees
- moved 220 16.0 mm to (60.0, 4.06)
- moved C2 5.60 mm to (9.71, 32.4)
- moved U$1 4.52 mm to (32.2, 35.4)
- moved U$2 2.86 mm to (53.5, 30.9)
Connections:
- removed net VSS: LCD1.1
- new net SCL: LCD1.4, NODE1.D1
- new net SDA: LCD1.3, NODE1.D2
- net GND: now also LCD1.1
Routing:
- net VCC: track 36.9 -> 233.2 mm
- net SCL: track 0.00 -> 68.3 mm
- net SDA: track 0.00 -> 58.4 mm
- net N$7: track 195.4 -> 167.0 mm
- net N$9: track 24.1 -> 33.2 mm
- net N$21: track 132.7 -> 139.1 mm
- net TX: track 81.8 -> 79.2 mm
- net RX: track 80.1 -> 77.6 mm
- net 3V: track 65.7 -> 63.4 mm
- net GND: track 69.3 -> 68.2 mm

Commit message: 143
Parts:
- added X1, X3: (no value), ak5002:AK500/2-H
- moved NODE1 2.25 mm to (35.0, 67.3)
Connections:
- new net D3: NODE1.D3, X1.2
- new net D4: NODE1.D4, X3.2
- net GND: now also X1.1, X3.1
Routing:
- net GND: track 68.2 -> 240.7 mm
- net N$7: track 167.0 -> 96.2 mm
- net D3: track 0.00 -> 57.4 mm
- net D4: track 0.00 -> 48.8 mm
- net SDA: track 58.4 -> 62.4 mm
- net SCL: track 68.3 -> 72.3 mm
- net TX: track 79.2 -> 83.2 mm
- net RX: track 77.6 -> 81.5 mm
- net VCC: track 233.2 -> 230.9 mm
- net N$21: track 139.1 -> 137.5 mm
- net 3V: track 63.4 -> 65.0 mm

Commit message: 447
Parts:
- added 1: KF76, kf76:KF76
- moved 220 8.84 mm to (67.9, 8.00)
Connections:
- new net N$2: 1.P$1, U$2.P$1
- net N$21: now also U$2.P$2
- net N$9: now also 1.P$2
Routing:
- net N$2: track 0.00 -> 116.7 mm
- net N$7: track 96.2 -> 152.1 mm
- net N$21: track 137.5 -> 93.6 mm
- net N$9: track 33.2 -> 48.0 mm
- net SDA: track 62.4 -> 64.7 mm
- net SCL: track 72.3 -> 74.4 mm

Commit message: 2158
Parts:
- removed NODE1: NODEMCU_ESP8266, nodemcu_esp8266:NODEMCU_ESP8266
- U$5: value SAPCER -> ESP32DEVKITV1; device spacer:SPACER -> ESP32-DEVKITV1:ESP32-DEVKITV1
- moved U$5 39.2 mm to (34.3, 58.9)
- moved U$8 24.5 mm to (67.7, 27.7), turned to 180 degrees
- moved U$2 16.8 mm to (56.6, 47.5)
- moved U$7 13.5 mm to (33.5, 78.1)
- moved X2 13.3 mm to (20.6, 84.3)
- moved U$3 13.0 mm to (36.5, 81.1)
- moved U$4 13.0 mm to (8.70, 9.43)
- moved U$6 12.8 mm to (3.52, 85.7), turned to 90 degrees
- moved U$1 8.29 mm to (28.9, 27.8)
- moved PZEM 7.65 mm to (12.9, 2.11)
- moved C1 7.65 mm to (37.5, 7.80)
- moved R3 7.65 mm to (31.3, 7.79)
- moved C2 6.68 mm to (3.90, 35.7)
- moved LCD1 3.07 mm to (11.6, 40.4)
- moved 1 2.12 mm to (50.2, 8.04)
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Connections:
- removed net 3V3: NODE1.3V3@2, NODE1.3V3@3
- net 3V: now also U$5.1; no longer NODE1.3V3@1
- net D3: now also U$5.12; no longer NODE1.D3
- net D4: now also U$5.11; no longer NODE1.D4
- net GND: now also U$5.28; no longer NODE1.GND@1, NODE1.GND@2, NODE1.GND@3, NODE1.GND@4
- net RX: now also U$5.7; no longer NODE1.D6
- net SCL: now also U$5.14; no longer NODE1.D1
- net SDA: now also U$5.13; no longer NODE1.D2
- net TX: now also U$5.8; no longer NODE1.D5
- net VCC: now also U$5.30; no longer NODE1.VIN
Routing:
- net N$7: track 152.1 -> 60.1 mm
- net VCC: track 230.9 -> 279.1 mm
- net 3V: track 65.0 -> 101.6 mm
- net SCL: track 74.4 -> 55.8 mm
- net SDA: track 64.7 -> 50.6 mm
- net GND: track 240.7 -> 252.4 mm
- net N$21: track 93.6 -> 105.3 mm
- net D4: track 48.8 -> 58.4 mm
- net D3: track 57.4 -> 65.3 mm
- net RX: track 81.5 -> 87.6 mm
- net N$9: track 48.0 -> 43.5 mm
- net TX: track 83.2 -> 87.6 mm
- net N$2: track 116.7 -> 116.1 mm
- removed copper zone on layer 16, net N$1
Other:
- board size 100 x 100 mm -> 90 x 90 mm

Commit message: 030
Parts:
- added BME280: BMP180, bme280:BPM180
- moved X3 13.3 mm to (52.8, 83.7)
- moved X1 13.1 mm to (63.1, 83.7)
- moved U$2 3.81 mm to (56.6, 43.6)
Connections:
- net GND: now also BME280.P$2
- net SCL: now also BME280.P$3
- net SDA: now also BME280.P$4
- net VCC: now also BME280.P$1
Routing:
- net VCC: track 279.1 -> 209.6 mm
- net SDA: track 50.6 -> 111.1 mm
- net SCL: track 55.8 -> 115.8 mm
- net GND: track 252.4 -> 238.7 mm
- net D3: track 65.3 -> 56.1 mm
- net D4: track 58.4 -> 51.3 mm
- net TX: track 87.6 -> 83.4 mm
- net N$21: track 105.3 -> 101.5 mm
- net N$2: track 116.1 -> 113.9 mm

Commit message: 033
Parts:
- moved U$2 2.12 mm to (56.7, 45.8)
Routing:
- net N$21: track 101.5 -> 103.7 mm
- net GND: track 238.7 -> 240.8 mm
- net N$2: track 113.9 -> 115.9 mm
Changed lines of the file:
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@@
 <attribute name="VALUE" x="1.627059375" y="38.586884375" size="1.27" layer="27" ratio="10"/>
 </element>
-<element name="U$2" library="TOROID" library_urn="urn:adsk.eagle:library:36786882" package="TOROID" package3d_urn="urn:adsk.eagle:package:36786885/2" value="TOROID" x="56.62823125" y="43.638421875" smashed="yes"/>
+<element name="U$2" library="TOROID" library_urn="urn:adsk.eagle:library:36786882" package="TOROID" package3d_urn="urn:adsk.eagle:package:36786885/2" value="TOROID" x="56.73400625" y="45.7543" smashed="yes"/>
 <element name="U$3" library="pzem30mmm" library_urn="urn:adsk.eagle:library:37023797" package="PZEM_FOOTPRINT" package3d_urn="urn:adsk.eagle:package:37023800/4" value="PZEM" x="36.51905" y="81.051696875" smashed="yes" rot="R180"/>
 <element name="U$4" library="spacer" library_urn="urn:adsk.eagle:library:37023739" package="SPACER" package3d_urn="urn:adsk.eagle:package:37023742/2" value="SAPCER" x="8.70009375" y="9.4327625" smashed="yes"/>
@@
 <contactref element="X2" pad="1"/>
 <wire x1="7.80196875" y1="29.015275" x2="7.74776875" y2="28.961075" width="0.8128" layer="16"/>
-<wire x1="7.74776875" y1="28.961075" x2="4.936371875" y2="28.961075" width="0.8128" layer="16"/>
-<wire x1="4.936371875" y1="28.961075" x2="3.43783125" y2="27.462534375" width="0.8128" layer="16"/>
-<wire x1="3.43783125" y1="27.462534375" x2="3.43783125" y2="19.48370625" width="0.8128" layer="16"/>
+<wire x1="3.43783125" y1="29.137696875" x2="3.43783125" y2="19.48370625" width="0.8128" layer="16"/>
 <wire x1="3.43783125" y1="19.48370625" x2="4.184303125" y2="18.737234375" width="0.8128" layer="16"/>
 <wire x1="4.184303125" y1="18.737234375" x2="12.170275" y2="18.737234375" width="0.8128" layer="16"/>
 <wire x1="3.89783125" y1="34.687796875" x2="3.43783125" y2="34.227796875" width="0.8128" layer="16"/>
-<wire x1="3.43783125" y1="34.227796875" x2="3.43783125" y2="27.462534375" width="0.8128" layer="16"/>
+<wire x1="3.43783125" y1="34.227796875" x2="3.43783125" y2="29.137696875" width="0.8128" layer="16"/>
 <wire x1="24.362940625" y1="84.2579" x2="24.4227625" y2="84.317721875" width="0.8128" layer="16"/>
 <contactref element="U$5" pad="28"/>
@@
 <wire x1="84.01016875" y1="80.9797875" x2="84.01016875" y2="78.294309375" width="0.8128" layer="16"/>
 <wire x1="84.01016875" y1="78.294309375" x2="77.331021875" y2="71.6151625" width="0.8128" layer="16"/>
-<wire x1="14.806234375" y1="86.83914375" x2="50.210265625" y2="86.83914375" width="0.8128" layer="16"/>
+<wire x1="14.806234375" y1="86.83914375" x2="24.3852875" y2="86.83914375" width="0.8128" layer="16"/>
+<wire x1="24.3852875" y1="86.83914375" x2="50.210265625" y2="86.83914375" width="0.8128" layer="16"/>
 <wire x1="50.210265625" y1="86.83914375" x2="60.490978125" y2="86.83914375" width="0.8128" layer="16"/>
 <wire x1="60.490978125" y1="86.83914375" x2="81.76333125" y2="86.83914375" width="0.8128" layer="16"/>
@@
 <wire x1="50.26134375" y1="83.709334375" x2="50.26134375" y2="86.788065625" width="0.8128" layer="16"/>
 <wire x1="50.26134375" y1="86.788065625" x2="50.210265625" y2="86.83914375" width="0.8128" layer="16"/>
-<wire x1="14.00058125" y1="70.169096875" x2="24.362940625" y2="84.2579" width="0" layer="19" extent="1-1"/>
+<wire x1="7.80196875" y1="29.015275" x2="3.560253125" y2="29.015275" width="0.8128" layer="16"/>
+<wire x1="3.560253125" y1="29.015275" x2="3.43783125" y2="29.137696875" width="0.8128" layer="16"/>
+<wire x1="24.362940625" y1="84.2579" x2="24.362940625" y2="86.816796875" width="0.8128" layer="16"/>
+<wire x1="24.362940625" y1="86.816796875" x2="24.3852875" y2="86.83914375" width="0.8128" layer="16"/>
 </signal>
 <signal name="TX">
@@
 <contactref element="PZEM" pad="P$1"/>
 <contactref element="U$2" pad="P$2"/>
-<wire x1="71.62823125" y1="37.558421875" x2="71.623259375" y2="37.55345" width="2.54" layer="16"/>
+<wire x1="71.73400625" y1="39.6743" x2="71.623259375" y2="39.563553125" width="2.54" layer="16"/>
 <wire x1="41.4630625" y1="27.455540625" x2="41.4630625" y2="15.529059375" width="2.54" layer="16"/>
 <wire x1="41.4630625" y1="15.529059375" x2="37.54625625" y2="11.612253125" width="2.54" layer="16"/>
@@
 <wire x1="67.6789" y1="16.255715625" x2="67.6789" y2="30.825396875" width="2.54" layer="16"/>
 <wire x1="67.6789" y1="30.459821875" x2="67.6789" y2="33.132153125" width="2.54" layer="16"/>
-<wire x1="71.623259375" y1="37.0765125" x2="71.623259375" y2="37.55345" width="2.54" layer="16"/>
+<wire x1="71.623259375" y1="37.0765125" x2="71.623259375" y2="39.563553125" width="2.54" layer="16"/>
 <wire x1="67.6789" y1="33.132153125" x2="71.623259375" y2="37.0765125" width="2.54" layer="16"/>
 <wire x1="67.6789" y1="30.825396875" x2="45.8584375" y2="30.825396875" width="2.54" layer="16"/>
@@
 <wire x1="56.1122125" y1="2.3622" x2="79.967875" y2="2.3622" width="2.54" layer="16"/>
 <wire x1="79.967875" y1="2.3622" x2="87.6378" y2="10.032125" width="2.54" layer="16"/>
-<wire x1="87.6378" y1="64.688421875" x2="71.62823125" y2="64.688421875" width="2.54" layer="16"/>
-<wire x1="87.6378" y1="10.032125" x2="87.6378" y2="64.688421875" width="2.54" layer="16"/>
+<wire x1="87.6378" y1="66.8043" x2="71.73400625" y2="66.8043" width="2.54" layer="16"/>
+<wire x1="87.6378" y1="10.032125" x2="87.6378" y2="66.8043" width="2.54" layer="16"/>
 </signal>
 </signals>

Commit message: 043
Parts:
- removed X1, X3: (no value), ak5002:AK500/2-H
- added P1, P2: (no value), ak5002:AK500/2-H
Connections:
- net D3: now also P1.2; no longer X1.2
- net D4: now also P2.2; no longer X3.2
- net GND: now also P1.1, P2.1; no longer X1.1, X3.1
Routing:
- net GND: track 240.8 -> 246.2 mm
- net D3: track 56.1 -> 53.2 mm
- net D4: track 51.3 -> 48.4 mm
Other:
- board text added: "SCL"
- board text added: "SDA"
