File: untitled.sch (EAGLE design)
At the start: 23 parts, among them K1 SLA-12VDC-SL-C, T1 BC547, X2 pzem-004t

Commit message: comit
comit
Parts:
- removed D1: 1N4004, diode:1N4004
- removed K1: SLA-12VDC-SL-C, SLA-12VDC-SL-C:SLA-12VDC-SL-C
- removed LED1: (no value), led:LED5MM
- removed OK1: PC817, optocoupler:PC817
- removed R1: 1k, rcl:R-EU_0207/15
- removed R2: 330, rcl:R-EU_0207/15
- removed RELAY: KF76, kf76:KF76
- removed T1: BC547, transistor:BC547
- added LCD1: LCD_2X16_SIL, lcd_2x16_led_backlight:LCD_2X16_SIL
Connections:
- removed net N$11: K1.NC, RELAY.P$2
- removed net N$18: LED1.A, R2.1
- removed net N$19: OK1.C, R2.2
- removed net N$2: OK1.EMIT, R1.1
- removed net N$20: LED1.C, NODE1.D7
- removed net N$3: R1.2, T1.B
- removed net N$5: D1.A, K1.COIL2, T1.C
- removed net N$8: K1.COM
- net 3V: no longer NODE1.3V3@2, OK1.A
- net GND: no longer T1.E
- net N$7: no longer RELAY.P$1
- net VCC: no longer D1.C, K1.COIL1, OK1.COL

Commit message: 0021
Connections:
- new net SCL: LCD1.SCL, NODE1.D1
- new net SDA: LCD1.SDA, NODE1.D2
- net GND: now also LCD1.GND
- net VCC: now also LCD1.VCC
Other:
- moved on the sheet: NODE1
Changed lines of the file:
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@@
 <attribute name="SHEET" x="230.505" y="5.08" size="2.54" layer="94"/>
 </instance>
-<instance part="NODE1" gate="G$1" x="58.42" y="86.36" smashed="yes">
-<attribute name="VALUE" x="48.26" y="58.42" size="1.27" layer="96"/>
-<attribute name="NAME" x="48.26" y="104.14" size="1.27" layer="95"/>
+<instance part="NODE1" gate="G$1" x="66.04" y="99.06" smashed="yes">
+<attribute name="VALUE" x="55.88" y="71.12" size="1.27" layer="96"/>
+<attribute name="NAME" x="55.88" y="116.84" size="1.27" layer="95"/>
 </instance>
 <instance part="X2" gate="-1" x="134.62" y="109.22" smashed="yes">
@@
 <instance part="220" gate="G$1" x="223.52" y="139.7" smashed="yes"/>
 <instance part="PZEM" gate="G$1" x="174.39433125" y="145.571615625" smashed="yes"/>
-<instance part="LCD1" gate="G$1" x="119.38" y="86.36" smashed="yes">
-<attribute name="NAME" x="111.76" y="43.18" size="1.27" layer="95"/>
+<instance part="LCD1" gate="G$1" x="142.24" y="83.82" smashed="yes">
+<attribute name="NAME" x="134.62" y="40.64" size="1.27" layer="95"/>
 </instance>
 </instances>
@@
 </segment>
 <segment>
-<label x="30.48" y="91.44" size="1.778" layer="95" rot="R180" xref="yes"/>
+<label x="38.1" y="104.14" size="1.778" layer="95" rot="R180" xref="yes"/>
 <pinref part="NODE1" gate="G$1" pin="D5"/>
-<wire x1="33.02" y1="91.44" x2="30.48" y2="91.44" width="0.1524" layer="91"/>
-<wire x1="43.18" y1="81.28" x2="33.02" y2="81.28" width="0.1524" layer="91"/>
-<wire x1="33.02" y1="81.28" x2="33.02" y2="91.44" width="0.1524" layer="91"/>
+<wire x1="40.64" y1="104.14" x2="38.1" y2="104.14" width="0.1524" layer="91"/>
+<wire x1="50.8" y1="93.98" x2="40.64" y2="93.98" width="0.1524" layer="91"/>
+<wire x1="40.64" y1="93.98" x2="40.64" y2="104.14" width="0.1524" layer="91"/>
 </segment>
 </net>
@@
 </segment>
 <segment>
-<label x="22.86" y="93.98" size="1.778" layer="95" rot="R180" xref="yes"/>
+<label x="30.48" y="106.68" size="1.778" layer="95" rot="R180" xref="yes"/>
 <pinref part="NODE1" gate="G$1" pin="D6"/>
-<wire x1="35.56" y1="93.98" x2="22.86" y2="93.98" width="0.1524" layer="91"/>
-<wire x1="43.18" y1="83.82" x2="35.56" y2="83.82" width="0.1524" layer="91"/>
-<wire x1="35.56" y1="83.82" x2="35.56" y2="93.98" width="0.1524" layer="91"/>
+<wire x1="43.18" y1="106.68" x2="30.48" y2="106.68" width="0.1524" layer="91"/>
+<wire x1="50.8" y1="96.52" x2="43.18" y2="96.52" width="0.1524" layer="91"/>
+<wire x1="43.18" y1="96.52" x2="43.18" y2="106.68" width="0.1524" layer="91"/>
 </segment>
 </net>
@@
 <segment>
 <pinref part="NODE1" gate="G$1" pin="VIN"/>
-<wire x1="73.66" y1="99.06" x2="76.2" y2="99.06" width="0.1524" layer="91"/>
+<wire x1="81.28" y1="111.76" x2="83.82" y2="111.76" width="0.1524" layer="91"/>
+<label x="83.82" y="111.76" size="1.778" layer="95" xref="yes"/>
 </segment>
 <segment>
@@
 <label x="22.86" y="157.48" size="1.778" layer="95" rot="R180" xref="yes"/>
 </segment>
+<segment>
+<pinref part="LCD1" gate="G$1" pin="VCC"/>
+<wire x1="129.54" y1="81.28" x2="109.22" y2="81.28" width="0.1524" layer="91"/>
+<label x="109.22" y="81.28" size="1.778" layer="95" rot="R180" xref="yes"/>
+</segment>
 </net>
 <net name="3V" class="0">
@@
 <segment>
 <pinref part="NODE1" gate="G$1" pin="3V3@1"/>
-<wire x1="43.18" y1="99.06" x2="38.1" y2="99.06" width="0.1524" layer="91"/>
-<label x="38.1" y="99.06" size="1.778" layer="95" rot="R180" xref="yes"/>
+<wire x1="50.8" y1="111.76" x2="45.72" y2="111.76" width="0.1524" layer="91"/>
+<label x="45.72" y="111.76" size="1.778" layer="95" rot="R180" xref="yes"/>
 </segment>
 </net>
@@
 <pinref part="NODE1" gate="G$1" pin="GND@4"/>
 <pinref part="X2" gate="-1" pin="S"/>
-<wire x1="132.08" y1="109.22" x2="93.98" y2="109.22" width="0.1524" layer="91"/>
-<wire x1="93.98" y1="109.22" x2="93.98" y2="96.52" width="0.1524" layer="91"/>
-<wire x1="93.98" y1="96.52" x2="73.66" y2="96.52" width="0.1524" layer="91"/>
+<wire x1="132.08" y1="109.22" x2="81.28" y2="109.22" width="0.1524" layer="91"/>
+</segment>
+<segment>
+<pinref part="LCD1" gate="G$1" pin="GND"/>
+<wire x1="129.54" y1="83.82" x2="101.6" y2="83.82" width="0.1524" layer="91"/>
+<label x="101.6" y="83.82" size="1.778" layer="95" rot="R180" xref="yes"/>
 </segment>
 </net>
@@
 </segment>
 </net>
+<net name="SDA" class="0">
+<segment>
+<pinref part="LCD1" gate="G$1" pin="SDA"/>
+<wire x1="129.54" y1="78.74" x2="116.84" y2="78.74" width="0.1524" layer="91"/>
+<label x="116.84" y="78.74" size="1.778" layer="95" rot="R180" xref="yes"/>
+</segment>
+<segment>
+<pinref part="NODE1" gate="G$1" pin="D2"/>
+<wire x1="50.8" y1="81.28" x2="35.56" y2="81.28" width="0.1524" layer="91"/>
+<label x="35.56" y="81.28" size="1.778" layer="95" rot="R180" xref="yes"/>
+</segment>
+</net>
+<net name="SCL" class="0">
+<segment>
+<pinref part="LCD1" gate="G$1" pin="SCL"/>
+<wire x1="129.54" y1="76.2" x2="124.46" y2="76.2" width="0.1524" layer="91"/>
+<label x="124.46" y="76.2" size="1.778" layer="95" rot="R180" xref="yes"/>
+</segment>
+<segment>
+<pinref part="NODE1" gate="G$1" pin="D1"/>
+<wire x1="50.8" y1="78.74" x2="48.26" y2="78.74" width="0.1524" layer="91"/>
+<label x="48.26" y="78.74" size="1.778" layer="95" rot="R180" xref="yes"/>
+</segment>
+</net>

Commit message: 143
Parts:
- added X1, X3: (no value), ak5002:AK500/2-H
Connections:
- new net D3: NODE1.D3, X1-2.KL
- new net D4: NODE1.D4, X3-2.KL
- net GND: now also X1-1.KL, X3-1.KL
Changed lines of the file:
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@@
 <part name="PZEM" library="kf76" library_urn="urn:adsk.eagle:library:37092210" deviceset="KF76" device="" package3d_urn="urn:adsk.eagle:package:37092213/3"/>
 <part name="LCD1" library="lcd_2x16_led_backlight" deviceset="LCD_2X16_SIL" device=""/>
+<part name="X1" library="ak5002" deviceset="AK500/2-H" device="" package3d_urn="urn:adsk.eagle:package:36988949/3"/>
+<part name="X3" library="ak5002" deviceset="AK500/2-H" device="" package3d_urn="urn:adsk.eagle:package:36988949/3"/>
 </parts>
 <sheets>
@@
 <instance part="LCD1" gate="G$1" x="142.24" y="83.82" smashed="yes">
 <attribute name="NAME" x="134.62" y="40.64" size="1.27" layer="95"/>
+</instance>
+<instance part="X1" gate="-1" x="203.2" y="83.82" smashed="yes" rot="R180">
+<attribute name="NAME" x="204.47" y="82.931" size="1.778" layer="95"/>
+</instance>
+<instance part="X1" gate="-2" x="203.2" y="88.9" smashed="yes" rot="R180">
+<attribute name="NAME" x="204.47" y="88.011" size="1.778" layer="95"/>
+<attribute name="VALUE" x="207.01" y="92.583" size="1.778" layer="96" rot="R180"/>
+</instance>
+<instance part="X3" gate="-1" x="203.2" y="68.58" smashed="yes" rot="R180">
+<attribute name="NAME" x="204.47" y="67.691" size="1.778" layer="95"/>
+</instance>
+<instance part="X3" gate="-2" x="203.2" y="73.66" smashed="yes" rot="R180">
+<attribute name="NAME" x="204.47" y="72.771" size="1.778" layer="95"/>
+<attribute name="VALUE" x="207.01" y="77.343" size="1.778" layer="96" rot="R180"/>
 </instance>
 </instances>
@@
 <label x="101.6" y="83.82" size="1.778" layer="95" rot="R180" xref="yes"/>
 </segment>
+<segment>
+<pinref part="X1" gate="-1" pin="KL"/>
+<wire x1="198.12" y1="83.82" x2="195.58" y2="83.82" width="0.1524" layer="91"/>
+<label x="195.58" y="83.82" size="1.778" layer="95" rot="R180" xref="yes"/>
+</segment>
+<segment>
+<pinref part="X3" gate="-1" pin="KL"/>
+<wire x1="198.12" y1="68.58" x2="195.58" y2="68.58" width="0.1524" layer="91"/>
+<label x="195.58" y="68.58" size="1.778" layer="95" rot="R180" xref="yes"/>
+</segment>
 </net>
 <net name="N$7" class="0">
@@
 </segment>
 </net>
+<net name="D3" class="0">
+<segment>
+<pinref part="NODE1" gate="G$1" pin="D3"/>
+<wire x1="50.8" y1="83.82" x2="48.26" y2="83.82" width="0.1524" layer="91"/>
+<label x="48.26" y="83.82" size="1.778" layer="95" rot="R180" xref="yes"/>
+</segment>
+<segment>
+<pinref part="X1" gate="-2" pin="KL"/>
+<wire x1="198.12" y1="88.9" x2="185.42" y2="88.9" width="0.1524" layer="91"/>
+<label x="185.42" y="88.9" size="1.778" layer="95" rot="R180" xref="yes"/>
+</segment>
+</net>
+<net name="D4" class="0">
+<segment>
+<pinref part="NODE1" gate="G$1" pin="D4"/>
+<wire x1="50.8" y1="86.36" x2="35.56" y2="86.36" width="0.1524" layer="91"/>
+<label x="35.56" y="86.36" size="1.778" layer="95" rot="R180" xref="yes"/>
+</segment>
+<segment>
+<pinref part="X3" gate="-2" pin="KL"/>
+<wire x1="198.12" y1="73.66" x2="185.42" y2="73.66" width="0.1524" layer="91"/>
+<label x="185.42" y="73.66" size="1.778" layer="95" rot="R180" xref="yes"/>
+</segment>
+</net>

Commit message: 447
Parts:
- added 1: KF76, kf76:KF76
Connections:
- new net N$2: 1.P$2, U$2.COM
- net N$21: now also U$2.L
- net N$9: now also 1.P$1
Changed lines of the file:
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@@
 <part name="X1" library="ak5002" deviceset="AK500/2-H" device="" package3d_urn="urn:adsk.eagle:package:36988949/3"/>
 <part name="X3" library="ak5002" deviceset="AK500/2-H" device="" package3d_urn="urn:adsk.eagle:package:36988949/3"/>
+<part name="1" library="kf76" library_urn="urn:adsk.eagle:library:37092210" deviceset="KF76" device="" package3d_urn="urn:adsk.eagle:package:37092213/3"/>
 </parts>
 <sheets>
@@
 <attribute name="VALUE" x="207.01" y="77.343" size="1.778" layer="96" rot="R180"/>
 </instance>
+<instance part="1" gate="G$1" x="215.9" y="116.84" smashed="yes"/>
 </instances>
 <busses>
@@
 <wire x1="198.12" y1="124.46" x2="170.18" y2="124.46" width="0.1524" layer="91"/>
 <wire x1="170.18" y1="124.46" x2="162.56" y2="124.46" width="0.1524" layer="91"/>
-<wire x1="162.56" y1="154.94" x2="162.56" y2="124.46" width="0.1524" layer="91"/>
+<wire x1="162.56" y1="154.94" x2="162.56" y2="149.86" width="0.1524" layer="91"/>
+<wire x1="162.56" y1="149.86" x2="162.56" y2="124.46" width="0.1524" layer="91"/>
 <wire x1="198.12" y1="139.7" x2="198.12" y2="124.46" width="0.1524" layer="91"/>
 <wire x1="220.98" y1="129.54" x2="203.2" y2="129.54" width="0.1524" layer="91"/>
@@
 <wire x1="170.18" y1="143.031615625" x2="170.18" y2="124.46" width="0.1524" layer="91"/>
 <junction x="170.18" y="124.46"/>
+<pinref part="U$2" gate="G$1" pin="L"/>
+<wire x1="162.56" y1="149.86" x2="144.78" y2="149.86" width="0.1524" layer="91"/>
+<junction x="162.56" y="149.86"/>
 </segment>
 </net>
@@
 <pinref part="U$8" gate="G$1" pin="IN"/>
 <wire x1="220.98" y1="152.4" x2="218.44" y2="152.4" width="0.1524" layer="91"/>
+<wire x1="220.98" y1="142.24" x2="213.36" y2="142.24" width="0.1524" layer="91"/>
+<junction x="220.98" y="142.24"/>
+<wire x1="213.36" y1="142.24" x2="213.36" y2="119.38" width="0.1524" layer="91"/>
+<pinref part="1" gate="G$1" pin="P$1"/>
+<wire x1="213.36" y1="119.38" x2="215.9" y2="119.38" width="0.1524" layer="91"/>
 </segment>
 </net>
@@
 </segment>
 </net>
+<net name="N$2" class="0">
+<segment>
+<pinref part="U$2" gate="G$1" pin="COM"/>
+<wire x1="144.78" y1="127" x2="144.78" y2="114.3" width="0.1524" layer="91"/>
+<wire x1="144.78" y1="114.3" x2="203.2" y2="114.3" width="0.1524" layer="91"/>
+<wire x1="205.74" y1="114.3" x2="203.2" y2="114.3" width="0.1524" layer="91"/>
+<pinref part="1" gate="G$1" pin="P$2"/>
+<wire x1="205.74" y1="114.3" x2="215.9" y2="114.3" width="0.1524" layer="91"/>
+</segment>
+</net>

Commit message: 2158
Parts:
- removed NODE1: NODEMCU_ESP8266, nodemcu_esp8266:NODEMCU_ESP8266
- U$5: value SAPCER -> ESP32DEVKITV1; device spacer:SAPCER -> ESP32-DEVKITV1:ESP32DEVKITV1
Connections:
- net 3V: now also U$5.3V3; no longer NODE1.3V3@1
- net D3: now also U$5.IO3; no longer NODE1.D3
- net D4: now also U$5.IO21; no longer NODE1.D4
- net GND: now also U$5.GND1; no longer NODE1.GND@4
- net RX: now also U$5.IO17; no longer NODE1.D6
- net SCL: now also U$5.IO22; no longer NODE1.D1
- net SDA: now also U$5.IO1; no longer NODE1.D2
- net TX: now also U$5.IO5; no longer NODE1.D5
- net VCC: now also U$5.VIN; no longer NODE1.VIN
Other:
- moved on the sheet: X1-1, X1-2, X3-1, X3-2

Commit message: 030
Parts:
- added BME280: BMP180, bme280:BMP180
Connections:
- net GND: now also BME280.GND
- net SCL: now also BME280.SCL
- net SDA: now also BME280.SDA
- net VCC: now also BME280.VCC
Changed lines of the file:
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@@
 <part name="1" library="kf76" library_urn="urn:adsk.eagle:library:37092210" deviceset="KF76" device="" package3d_urn="urn:adsk.eagle:package:37092213/3"/>
 <part name="U$5" library="ESP32-DEVKITV1" deviceset="ESP32DEVKITV1" device=""/>
+<part name="BME280" library="bme280" deviceset="BMP180" device=""/>
 </parts>
 <sheets>
@@
 <attribute name="NAME" x="63.5" y="102.87" size="1.27" layer="95"/>
 </instance>
+<instance part="BME280" gate="G$1" x="223.52" y="55.88" smashed="yes"/>
 </instances>
 <busses>
@@
 <wire x1="76.2" y1="99.06" x2="81.28" y2="99.06" width="0.1524" layer="91"/>
 <label x="81.28" y="99.06" size="1.778" layer="95" xref="yes"/>
+</segment>
+<segment>
+<pinref part="BME280" gate="G$1" pin="VCC"/>
+<wire x1="208.28" y1="68.58" x2="195.58" y2="68.58" width="0.1524" layer="91"/>
+<label x="195.58" y="68.58" size="1.778" layer="95" rot="R180" xref="yes"/>
 </segment>
 </net>
@@
 <label x="93.98" y="96.52" size="1.778" layer="95" xref="yes"/>
 </segment>
+<segment>
+<pinref part="BME280" gate="G$1" pin="GND"/>
+<wire x1="208.28" y1="63.5" x2="195.58" y2="63.5" width="0.1524" layer="91"/>
+<label x="195.58" y="63.5" size="1.778" layer="95" rot="R180" xref="yes"/>
+</segment>
 </net>
 <net name="N$7" class="0">
@@
 <label x="22.86" y="68.58" size="1.778" layer="95" rot="R180" xref="yes"/>
 </segment>
+<segment>
+<pinref part="BME280" gate="G$1" pin="SDA"/>
+<wire x1="208.28" y1="53.34" x2="195.58" y2="53.34" width="0.1524" layer="91"/>
+<label x="195.58" y="53.34" size="1.778" layer="95" rot="R180" xref="yes"/>
+</segment>
 </net>
 <net name="SCL" class="0">
@@
 <label x="33.02" y="66.04" size="1.778" layer="95" rot="R180" xref="yes"/>
 </segment>
-</net>
+<segment>
+<pinref part="BME280" gate="G$1" pin="SCL"/>
+<wire x1="208.28" y1="58.42" x2="195.58" y2="58.42" width="0.1524" layer="91"/>
+<label x="195.58" y="58.42" size="1.778" layer="95" rot="R180" xref="yes"/>
+</segment>
+</net>

Commit message: 043
Parts:
- renumbered X1 to P1, X3 to P2
Changed lines of the file:
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@@
 <part name="PZEM" library="kf76" library_urn="urn:adsk.eagle:library:37092210" deviceset="KF76" device="" package3d_urn="urn:adsk.eagle:package:37092213/3"/>
 <part name="LCD1" library="lcd_2x16_led_backlight" deviceset="LCD_2X16_SIL" device=""/>
-<part name="X1" library="ak5002" deviceset="AK500/2-H" device="" package3d_urn="urn:adsk.eagle:package:36988949/3"/>
-<part name="X3" library="ak5002" deviceset="AK500/2-H" device="" package3d_urn="urn:adsk.eagle:package:36988949/3"/>
+<part name="P1" library="ak5002" deviceset="AK500/2-H" device="" package3d_urn="urn:adsk.eagle:package:36988949/3"/>
+<part name="P2" library="ak5002" deviceset="AK500/2-H" device="" package3d_urn="urn:adsk.eagle:package:36988949/3"/>
 <part name="1" library="kf76" library_urn="urn:adsk.eagle:library:37092210" deviceset="KF76" device="" package3d_urn="urn:adsk.eagle:package:37092213/3"/>
 <part name="U$5" library="ESP32-DEVKITV1" deviceset="ESP32DEVKITV1" device=""/>
@@
 <attribute name="NAME" x="134.62" y="40.64" size="1.27" layer="95"/>
 </instance>
-<instance part="X1" gate="-1" x="180.34" y="99.06" smashed="yes" rot="R180">
+<instance part="P1" gate="-1" x="180.34" y="99.06" smashed="yes" rot="R180">
 <attribute name="NAME" x="181.61" y="98.171" size="1.778" layer="95"/>
 </instance>
-<instance part="X1" gate="-2" x="180.34" y="104.14" smashed="yes" rot="R180">
+<instance part="P1" gate="-2" x="180.34" y="104.14" smashed="yes" rot="R180">
 <attribute name="NAME" x="181.61" y="103.251" size="1.778" layer="95"/>
 <attribute name="VALUE" x="184.15" y="107.823" size="1.778" layer="96" rot="R180"/>
 </instance>
-<instance part="X3" gate="-1" x="180.34" y="83.82" smashed="yes" rot="R180">
+<instance part="P2" gate="-1" x="180.34" y="83.82" smashed="yes" rot="R180">
 <attribute name="NAME" x="181.61" y="82.931" size="1.778" layer="95"/>
 </instance>
-<instance part="X3" gate="-2" x="180.34" y="88.9" smashed="yes" rot="R180">
+<instance part="P2" gate="-2" x="180.34" y="88.9" smashed="yes" rot="R180">
 <attribute name="NAME" x="181.61" y="88.011" size="1.778" layer="95"/>
 <attribute name="VALUE" x="184.15" y="92.583" size="1.778" layer="96" rot="R180"/>
@@
 </segment>
 <segment>
-<pinref part="X1" gate="-1" pin="KL"/>
+<pinref part="P1" gate="-1" pin="KL"/>
 <wire x1="175.26" y1="99.06" x2="172.72" y2="99.06" width="0.1524" layer="91"/>
 <label x="172.72" y="99.06" size="1.778" layer="95" rot="R180" xref="yes"/>
 </segment>
 <segment>
-<pinref part="X3" gate="-1" pin="KL"/>
+<pinref part="P2" gate="-1" pin="KL"/>
 <wire x1="175.26" y1="83.82" x2="172.72" y2="83.82" width="0.1524" layer="91"/>
 <label x="172.72" y="83.82" size="1.778" layer="95" rot="R180" xref="yes"/>
@@
 <net name="D3" class="0">
 <segment>
-<pinref part="X1" gate="-2" pin="KL"/>
+<pinref part="P1" gate="-2" pin="KL"/>
 <wire x1="175.26" y1="104.14" x2="162.56" y2="104.14" width="0.1524" layer="91"/>
 <label x="162.56" y="104.14" size="1.778" layer="95" rot="R180" xref="yes"/>
@@
 <net name="D4" class="0">
 <segment>
-<pinref part="X3" gate="-2" pin="KL"/>
+<pinref part="P2" gate="-2" pin="KL"/>
 <wire x1="175.26" y1="88.9" x2="162.56" y2="88.9" width="0.1524" layer="91"/>
 <label x="162.56" y="88.9" size="1.778" layer="95" rot="R180" xref="yes"/>

Commit message: 213
Parts:
- added R1: 100, rcl:R-EU_0207/12
Connections:
- new net N$1: P2-2.KL, R1.2
- net D3: no longer P1-2.KL
- net D4: now also R1.1; no longer P2-2.KL
- net VCC: now also P1-2.KL
Changed lines of the file:
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@@
 <part name="U$5" library="ESP32-DEVKITV1" deviceset="ESP32DEVKITV1" device=""/>
 <part name="BME280" library="bme280" deviceset="BMP180" device=""/>
+<part name="R1" library="rcl" library_urn="urn:adsk.eagle:library:334" deviceset="R-EU_" device="0207/12" package3d_urn="urn:adsk.eagle:package:23489/1" value="100"/>
 </parts>
 <sheets>
@@
 </instance>
 <instance part="BME280" gate="G$1" x="223.52" y="55.88" smashed="yes"/>
+<instance part="R1" gate="G$1" x="165.1" y="88.9" smashed="yes">
+<attribute name="NAME" x="161.29" y="90.3986" size="1.778" layer="95"/>
+<attribute name="VALUE" x="161.29" y="85.598" size="1.778" layer="96"/>
+</instance>
 </instances>
 <busses>
@@
 <wire x1="208.28" y1="68.58" x2="195.58" y2="68.58" width="0.1524" layer="91"/>
 <label x="195.58" y="68.58" size="1.778" layer="95" rot="R180" xref="yes"/>
+</segment>
+<segment>
+<pinref part="P1" gate="-2" pin="KL"/>
+<wire x1="175.26" y1="104.14" x2="162.56" y2="104.14" width="0.1524" layer="91"/>
+<label x="162.56" y="104.14" size="1.778" layer="95" rot="R180" xref="yes"/>
 </segment>
 </net>
@@
 <net name="D3" class="0">
 <segment>
-<pinref part="P1" gate="-2" pin="KL"/>
-<wire x1="175.26" y1="104.14" x2="162.56" y2="104.14" width="0.1524" layer="91"/>
-<label x="162.56" y="104.14" size="1.778" layer="95" rot="R180" xref="yes"/>
-</segment>
-<segment>
 <pinref part="U$5" gate="G$1" pin="IO3"/>
 <wire x1="40.64" y1="71.12" x2="33.02" y2="71.12" width="0.1524" layer="91"/>
@@
 <net name="D4" class="0">
 <segment>
-<pinref part="P2" gate="-2" pin="KL"/>
-<wire x1="175.26" y1="88.9" x2="162.56" y2="88.9" width="0.1524" layer="91"/>
-<label x="162.56" y="88.9" size="1.778" layer="95" rot="R180" xref="yes"/>
+<label x="154.94" y="88.9" size="1.778" layer="95" rot="R180" xref="yes"/>
+<wire x1="160.02" y1="88.9" x2="154.94" y2="88.9" width="0.1524" layer="91"/>
+<pinref part="R1" gate="G$1" pin="1"/>
 </segment>
 <segment>
@@
 </segment>
 </net>
+<net name="N$1" class="0">
+<segment>
+<pinref part="P2" gate="-2" pin="KL"/>
+<wire x1="175.26" y1="88.9" x2="170.18" y2="88.9" width="0.1524" layer="91"/>
+<pinref part="R1" gate="G$1" pin="2"/>
+</segment>
+</net>
